File: kicad/dw-card.kicad_pcb (KiCad board)
At the start: 4 copper layers, 85.5 x 54 mm, 81 parts, among them J1 Conn_01x06, P1 USB_C_Plug_USB2.0, Q1 MMBT3904, Q2 MMBT3904, Q3 MMBT3904, SW1 PTS526, SW2 PTS526, SW3 PTS526, SW4 PTS526, SW5 PTS526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

Commit message: add gh qrcode & readme
Parts:
- added LDW3: Logo_Open_Hardware_Small, dw-card:qrcode_github, B.Cu at (148.7, 93.0)
Other:
- board text removed: "IoT Engineer Full-stack developer damien@weber.sx"

Commit message: invert A & B buttons
Parts:
- moved G3 12.0 mm to (182.5, 100.5)
- moved G4 12.0 mm to (170.5, 100.5)
Changed lines of the file:
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@@
   (net 78 "unconnected-(SW9-C-Pad3)")
   (footprint "dw-card:btn_b" (layer "F.Cu")
-    (at 182.5 100.5)
+    (at 170.5 100.5)
     (property "Sheetfile" "dw-card.kicad_sch")
     (property "Sheetname" "")
@@
   )
   (footprint "dw-card:btn_a" (layer "F.Cu")
-    (at 170.5 100.5)
+    (at 182.5 100.5)
     (property "Sheetfile" "dw-card.kicad_sch")
     (property "Sheetname" "")
