File: kicad/dw-card.kicad_sch (KiCad schematic)
At the start: 81 parts, among them J1 Conn_01x06, P1 USB_C_Plug_USB2.0, Q1 MMBT3904, Q2 MMBT3904, Q3 MMBT3904, SW1 PTS526, SW2 PTS526, SW3 PTS526, SW4 PTS526, SW5 PTS526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

Commit message: invert A & B buttons
Parts:
- added LDW3: Logo_Open_Hardware_Small, dw-card:qrcode_github, symbol Graphic:Logo_Open_Hardware_Small
Changed lines of the file:
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@@
+    )
+  )
+  (symbol (lib_id "Graphic:Logo_Open_Hardware_Small") (at 247.65 173.99 0) (unit 1)
+    (in_bom yes) (on_board yes) (dnp no) (fields_autoplaced)
+    (property "Reference" "LDW3" (at 247.65 167.005 0)
+      (effects (font (size 1.27 1.27)) hide)
+    )
+    (property "Value" "Logo_Open_Hardware_Small" (at 247.65 179.705 0)
+      (effects (font (size 1.27 1.27)) hide)
+    )
+    (property "Footprint" "dw-card:qrcode_github" (at 247.65 173.99 0)
+      (effects (font (size 1.27 1.27)) hide)
+    )
+    (property "Datasheet" "~" (at 247.65 173.99 0)
+      (effects (font (size 1.27 1.27)) hide)
+    )
+    (instances
+      (project "dw-card"
+        (path "/e63e39d7-6ac0-4ffd-8aa3-1841a4541b55"
+          (reference "LDW3") (unit 1)
+        )
+      )
     )
   )
